File: electronics/board/mini-dyno/mini-dyno.kicad_sch (KiCad schematic)
At the start: 44 parts, among them J1 Conn_01x04_Pin, J2 Conn_01x03_Pin, SW1 SW_Push, SW2 SW_Push, U1 ESP32-C3-MINI-1, U2 TLV75733PDBVR, U4 HX711_C6705483

Commit message: Update PCB
Parts:
- C11: footprint Capacitor_SMD:C_0805_2012Metric -> easyeda2kicad:CAP-TH_BD6.3-P2.50-D1.0-FD
Changed lines of the file:
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@@
 			)
 		)
-		(property "Footprint" "Capacitor_SMD:C_0805_2012Metric"
+		(property "Footprint" "easyeda2kicad:CAP-TH_BD6.3-P2.50-D1.0-FD"
 			(at 146.05 163.5252 0)
 			(effects

Commit message: Update PCB
Parts:
- removed C11: 100uF, easyeda2kicad:CAP-TH_BD6.3-P2.50-D1.0-FD, symbol Device:C
- added C11: 35ZLH100MEFC6.3X11, easyeda2kicad:CAP-TH_BD6.3-P2.50-D1.0-FD, symbol easyeda2kicad:35ZLH100MEFC6.3X11
Connections:
- net +5V: now also C11.1
- net GND: now also C11.2
Changed lines of the file:
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@@
 	)
 	(junction
-		(at 146.05 162.56)
-		(diameter 0)
-		(color 0 0 0 0)
-	)
-	(junction
 		(at 33.02 91.44)
 		(diameter 0)
@@
 	)
 	(junction
+		(at 146.05 162.56)
+		(diameter 0)
+		(color 0 0 0 0)
+	)
+	(junction
 		(at 194.31 137.16)
 		(diameter 0)
@@
 	(wire
 		(pts
-			(xy 146.05 162.56) (xy 146.05 168.91)
-		)
-		(stroke
-			(width 0)
-			(type default)
-		)
-	)
-	(wire
-		(pts
 			(xy 40.64 157.48) (xy 41.91 157.48)
 		)
@@
 	(wire
 		(pts
+			(xy 146.05 162.56) (xy 146.05 168.91)
+		)
+		(stroke
+			(width 0)
+			(type default)
+		)
+	)
+	(wire
+		(pts
 			(xy 90.17 151.13) (xy 102.87 151.13)
 		)
@@
 	)
 	(symbol
+		(lib_id "easyeda2kicad:35ZLH100MEFC6.3X11")
+		(at 149.86 162.56 0)
+		(unit 1)
+		(exclude_from_sim no)
+		(in_bom yes)
+		(on_board yes)
+		(dnp no)
+		(fields_autoplaced yes)
+		(property "Reference" "C11"
+			(at 149.255 156.21 0)
+			(effects
+				(font
+					(size 1.27 1.27)
+				)
+			)
+		)
+		(property "Value" "35ZLH100MEFC6.3X11"
+			(at 149.255 158.75 0)
+			(effects
+				(font
+					(size 1.27 1.27)
+				)
+			)
+		)
+		(property "Footprint" "easyeda2kicad:CAP-TH_BD6.3-P2.50-D1.0-FD"
+			(at 149.86 170.18 0)
+			(effects
+				(font
+					(size 1.27 1.27)
+				)
+				(hide yes)
+			)
+		)
+		(property "Datasheet" "https://lcsc.com/product-detail/Aluminum-Electrolytic-Capacitors-Leaded_Rubycon_35ZLH100MEFC6-3X1_100uF-107-20-35V_C109392.html"
+			(at 149.86 172.72 0)
+			(effects
+				(font
+					(size 1.27 1.27)
+				)
+				(hide yes)
+			)
+		)
+		(property "Description" ""
+			(at 149.86 162.56 0)
+			(effects
+				(font
+					(size 1.27 1.27)
+				)
+				(hide yes)
+			)
+		)
+		(property "LCSC Part" "C109392"
+			(at 149.86 175.26 0)
+			(effects
+				(font
+					(size 1.27 1.27)
+				)
+				(hide yes)
+			)
+		)
+		(pin "1"
+		)
+		(pin "2"
+		)
+		(instances
+			(project ""
+				(path "/2187563e-ed7c-448b-a062-1766b86d965d"
+					(reference "C11")
+					(unit 1)
+				)
+			)
+		)
+	)
+	(symbol
 		(lib_id "Device:R")
 		(at 204.47 53.34 90)
@@
 					(unit 1)
 				)
-			)
-		)
-	)
-	(symbol
-		(lib_id "Device:C")
-		(at 149.86 162.56 270)
-		(unit 1)
-		(exclude_from_sim no)
-		(in_bom yes)
-		(on_board yes)
-		(dnp no)
-		(property "Reference" "C11"
-			(at 156.464 157.988 90)
-			(effects
-				(font
-					(size 1.27 1.27)
-				)
-				(justify right)
-			)
-		)
-		(property "Value" "100uF"
-			(at 157.988 160.02 90)
-			(effects
-				(font
-					(size 1.27 1.27)
-				)
-				(justify right)
-			)
-		)
-		(property "Footprint" "easyeda2kicad:CAP-TH_BD6.3-P2.50-D1.0-FD"
-			(at 146.05 163.5252 0)
-			(effects
-				(font
-					(size 1.27 1.27)
-				)
-				(hide yes)
-			)
-		)
-		(property "Datasheet" "~"
-			(at 149.86 162.56 0)
-			(effects
-				(font
-					(size 1.27 1.27)
-				)
-				(hide yes)
-			)
-		)
-		(property "Description" "Unpolarized capacitor"
-			(at 149.86 162.56 0)
-			(effects
-				(font
-					(size 1.27 1.27)
-				)
-				(hide yes)
-			)
-		)
-		(pin "2"
-		)
-		(pin "1"
-		)
-		(instances
-			(project "mini-dyno"
-				(path "/2187563e-ed7c-448b-a062-1766b86d965d"
-					(reference "C11")
-					(unit 1)
-				)

Commit message: Update PCB
Parts:
- removed C11: 35ZLH100MEFC6.3X11, easyeda2kicad:CAP-TH_BD6.3-P2.50-D1.0-FD, symbol easyeda2kicad:35ZLH100MEFC6.3X11
- removed C5, C6: 10uF, Capacitor_SMD:C_0805_2012Metric, symbol Device:C
- removed D1: ESD122DMYR, easyeda2kicad:X2SON-3_L1.3-W0.6-L, symbol easyeda2kicad:ESD122DMYR
- removed D2: SMBJ5.0A_C83333, easyeda2kicad:SMB_L4.6-W3.6-LS5.3-RD, symbol easyeda2kicad:SMBJ5.0A_C83333
- removed D5: SS310_C14281, easyeda2kicad:SMB_L4.6-W3.6-LS5.3-RD, symbol easyeda2kicad:SS310_C14281
- removed F1: TLC-PSML400, easyeda2kicad:F0805, symbol easyeda2kicad:TLC-PSML400
- removed R4, R9: 5.1kΩ, Resistor_SMD:R_0805_2012Metric, symbol Device:R
- removed R5: 10kΩ, Resistor_SMD:R_0805_2012Metric, symbol Device:R
- removed U2: TLV75733PDBVR, easyeda2kicad:SOT-23-5_L2.9-W1.6-P0.95-LS2.8-BL, symbol easyeda2kicad:TLV75733PDBVR
- removed USB1, USB3: MC-710A, easyeda2kicad:USB-C-TH_MC-710A, symbol easyeda2kicad:MC-710A
- added C1, C10, C4: 10uF, Capacitor_SMD:C_0805_2012Metric, symbol Device:C
- added D1: D_TVS, Diode_SMD:D_SMB, symbol Device:D_Zener
- added D2: D_Schottky, Diode_SMD:D_SMB, symbol Device:D_Schottky
- added F1: Polyfuse, Fuse:Fuse_0805_2012Metric_Pad1.15x1.40mm_HandSolder, symbol Device:Polyfuse
- added H1, H2, H3, H4: (no value), MountingHole:MountingHole_3.2mm_M3_Pad, symbol Mechanical:MountingHole_Pad
- added Q1: AO3400A, Package_TO_SOT_SMD:SOT-23_Handsoldering, symbol Transistor_FET:Q_NMOS_DGS
- added R1, R19: 5.1kΩ, Resistor_SMD:R_0805_2012Metric, symbol Device:R
- added R11: 100Ω, Resistor_SMD:R_0805_2012Metric, symbol Device:R
- added R12: 10kΩ, Resistor_SMD:R_0805_2012Metric, symbol Device:R
- added R13, R3, R7: 0Ω, Resistor_SMD:R_1206_3216Metric_Pad1.30x1.75mm_HandSolder, symbol Device:R
- added TP1: VBUS, TestPoint:TestPoint_THTPad_2.0x2.0mm_Drill1.0mm, symbol Connector:TestPoint
- added TP2: 5V, TestPoint:TestPoint_THTPad_2.0x2.0mm_Drill1.0mm, symbol Connector:TestPoint
- added TP3: 3V3, TestPoint:TestPoint_THTPad_2.0x2.0mm_Drill1.0mm, symbol Connector:TestPoint
- added TP4: 5V_MOTOR, TestPoint:TestPoint_THTPad_2.0x2.0mm_Drill1.0mm, symbol Connector:TestPoint
- added TP5: GND, TestPoint:TestPoint_THTPad_2.0x2.0mm_Drill1.0mm, symbol Connector:TestPoint
- added U1: AZ1117IH-3.3TRG1, easyeda2kicad:SOT-223-4_L6.5-W3.5-P2.30-LS7.0-BR, symbol easyeda2kicad:AZ1117IH-3.3TRG1
- added U4: TPD2S017, Package_TO_SOT_SMD:SOT-23-6, symbol Power_Protection:TPD2S017
- added USB1: POWER, easyeda2kicad:USC-C-SMD_USB4085-GF-A, symbol easyeda2kicad:USB4085-GF-A_C7095263
- added USB2: DATA, easyeda2kicad:USC-C-SMD_USB4085-GF-A, symbol easyeda2kicad:USB4085-GF-A_C7095263
- R16: renamed from R12; value 100Ω -> 1kΩ
- R17: renamed from R14; value 100Ω -> 1kΩ
- R6: value 10kΩ -> 0Ω; footprint Resistor_SMD:R_0805_2012Metric -> Resistor_SMD:R_1206_3216Metric_Pad1.30x1.75mm_HandSolder
- U2: renamed from U4; value HX711_C6705483 -> HX711
- renumbered C12 to C11, C7 to C12, C9 to C2, C10 to C3, C8 to C5, C4 to C6, C1 to C7, C2 to C8, C3 to C9, R1 to R10, R13 to R14, R11 to R15, R3 to R18, R10 to R20, R15 to R4, R16 to R5, R7 to R9, U1 to U3
Connections:
- net +3V3: now also R6.2, R7.1, TP3.1; no longer C5.2, U2.1 (VSUP), U2.16 (DVDD)
- net +5V: now also D1.1 (K), F1.2, R13.2, R3.2, TP2.1, U4.5 (VCC); no longer C11.2, MOTOR1.1 (VCC)
- net GND: now also R20.2, C1.2, C10.1, C4.2, D1.2 (A), H1.1, H2.1, H3.1, H4.1, Q1.3 (S), R1.1, R12.1, R19.1, TP5.1, U1.1 (ADJ/GND), U4.2 (GND), USB1.A1 (GND), USB1.A12 (GND), USB1.B1 (GND), USB1.B12 (GND), USB2.A1 (GND), USB2.A12 (GND), USB2.B1 (GND), USB2.B12 (GND); no longer MOTOR1.4 (GND), R20.1
- net D+: now reaches U3.27 (GPIO19/USB_D+)
- net D+: now also U4.1 (CH1Out)
- net CC2_P: now reaches R2.2
- net CC2_P: now also USB1.B5 (CC2)
- net CC1: now reaches R18.2
- net CC1: now also USB2.A5 (CC1)
- net at R6.1: now also C5.2, U2.1 (VSUP), U2.16 (DVDD); no longer U3.26 (GPIO18/USB_D-)
- net FET_GATE: now reaches U3.30 (GPIO20/U0RXD)
- net FET_GATE: now also R11.1
- net at R8.2: now also USB1.S1
- new net: Q1.2 (G), R11.2, R12.2
- new net: C1.1, R3.1, U1.3 (INPUT)
- new net: C4.1, R7.2, U1.2 (OUTPUT), U1.4 (VOUT)
- new net: R20.1, USB2.S1
- new net: C10.2, C11.2, D2.1 (K), MOTOR1.1 (VCC), R13.1, TP4.1
- new net CC1_P: R1.2, USB1.A5 (CC1)
- new net CC2: R19.2, USB2.B5 (CC2)
- new net D-: U3.26 (GPIO18/USB_D-), U4.6 (CH2Out)
- new net ESD_D+: U4.3 (CH1In), USB2.A6 (Dp1), USB2.B7 (Dn2)
- new net ESD_D-: U4.4 (CH2Int), USB2.A7 (Dn1), USB2.B6 (Dp2)
- new net MOTOR_DRAIN: D2.2 (A), MOTOR1.4 (GND), Q1.1 (D)
- new net VBUS: F1.1, TP1.1, USB1.A4 (VBUS), USB1.A9 (VBUS), USB1.B4 (VBUS), USB1.B9 (VBUS)
Other:
- note added: "MOUNTING HOLES"
- moved on the sheet: C11, J2, MOTOR1, R14, R18, R20

Commit message: Update PCB Layout
Connections:
- net +3V3: now also U4.5 (VCC)
- net +5V: no longer U4.5 (VCC)
Changed lines of the file:
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@@
-	)
-	(symbol
-		(lib_id "power:+5V")
-		(at 215.9 21.59 0)
-		(unit 1)
-		(body_style 1)
-		(exclude_from_sim no)
-		(in_bom yes)
-		(on_board yes)
-		(in_pos_files yes)
-		(dnp no)
-		(fields_autoplaced yes)
-		(property "Reference" "#PWR039"
-			(at 215.9 25.4 0)
-			(hide yes)
-			(show_name no)
-			(do_not_autoplace no)
-			(effects
-				(font
-					(size 1.27 1.27)
-				)
-			)
-		)
-		(property "Value" "+5V"
-			(at 215.9 16.51 0)
-			(show_name no)
-			(do_not_autoplace no)
-			(effects
-				(font
-					(size 1.27 1.27)
-				)
-			)
-		)
-		(property "Footprint" ""
-			(at 215.9 21.59 0)
-			(hide yes)
-			(show_name no)
-			(do_not_autoplace no)
-			(effects
-				(font
-					(size 1.27 1.27)
-				)
-			)
-		)
-		(property "Datasheet" ""
-			(at 215.9 21.59 0)
-			(hide yes)
-			(show_name no)
-			(do_not_autoplace no)
-			(effects
-				(font
-					(size 1.27 1.27)
-				)
-			)
-		)
-		(property "Description" "Power symbol creates a global label with name \"+5V\""
-			(at 215.9 21.59 0)
-			(hide yes)
-			(show_name no)
-			(do_not_autoplace no)
-			(effects
-				(font
-					(size 1.27 1.27)
-				)
-			)
-		)
-		(pin "1"
-		)
-		(instances
-			(project "mini-dyno"
-				(path "/2187563e-ed7c-448b-a062-1766b86d965d"
-					(reference "#PWR039")
-					(unit 1)
-				)
-			)
-		)
 	)
 	(symbol
@@
 					(unit 1)
 				)
+			)
+		)
+	)
+	(symbol
+		(lib_id "power:+3V3")
+		(at 215.9 21.59 0)
+		(unit 1)
+		(body_style 1)
+		(exclude_from_sim no)
+		(in_bom yes)
+		(on_board yes)
+		(in_pos_files yes)
+		(dnp no)
+		(fields_autoplaced yes)
+		(property "Reference" "#PWR019"
+			(at 215.9 25.4 0)
+			(hide yes)
+			(show_name no)
+			(do_not_autoplace no)
+			(effects
+				(font
+					(size 1.27 1.27)
+				)
+			)
+		)
+		(property "Value" "+3V3"
+			(at 215.9 16.51 0)
+			(show_name no)
+			(do_not_autoplace no)
+			(effects
+				(font
+					(size 1.27 1.27)
+				)
+			)
+		)
+		(property "Footprint" ""
+			(at 215.9 21.59 0)
+			(hide yes)
+			(show_name no)
+			(do_not_autoplace no)
+			(effects
+				(font
+					(size 1.27 1.27)
+				)
+			)
+		)
+		(property "Datasheet" ""
+			(at 215.9 21.59 0)
+			(hide yes)
+			(show_name no)
+			(do_not_autoplace no)
+			(effects
+				(font
+					(size 1.27 1.27)
+				)
+			)
+		)
+		(property "Description" "Power symbol creates a global label with name \"+3V3\""
+			(at 215.9 21.59 0)
+			(hide yes)
+			(show_name no)
+			(do_not_autoplace no)
+			(effects
+				(font
+					(size 1.27 1.27)
+				)
+			)
+		)
+		(pin "1"
+		)
+		(instances
+			(project "mini-dyno"
+				(path "/2187563e-ed7c-448b-a062-1766b86d965d"
+					(reference "#PWR019")
+					(unit 1)
+				)
