File: electronics/board/mini-dyno/mini-dyno.kicad_pcb (KiCad board)
At the start: 2 copper layers, 65 x 37 mm, 44 parts, among them J1 Conn_01x04_Pin, J2 Conn_01x03_Pin, SW1 SW_Push, SW2 SW_Push, U1 ESP32-C3-MINI-1, U2 TLV75733PDBVR, U4 HX711_C6705483

Commit message: Update PCB
Parts:
- C11: footprint Capacitor_SMD:C_0805_2012Metric -> easyeda2kicad:CAP-TH_BD6.3-P2.50-D1.0-FD
- moved C12 2.20 mm to (178.2, 95.0)
- moved D5 2.00 mm to (178.2, 100.0)
- renumbered POWER to D3, STATUS to D4
Routing:
- net +5V: track 39.1 -> 42.6 mm
Changed lines of the file:
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@@
 		(25 "Edge.Cuts" user)
 		(27 "Margin" user)
-		(31 "F.CrtYd" user)
-		(29 "B.CrtYd" user)
+		(31 "F.CrtYd" user "F.Courtyard")
+		(29 "B.CrtYd" user "B.Courtyard")
 		(35 "F.Fab" user)
 	)
@@
 	(footprint "easyeda2kicad:SMB_L4.6-W3.6-LS5.3-RD"
 		(layer "F.Cu")
-		(at 178.2 98 -90)
+		(at 178.2 100 -90)
 		(property "Reference" "D5"
 			(at 0 2.9 90)
@@
 		)
 	)
-	(footprint "Capacitor_SMD:C_0805_2012Metric"
+	(footprint "easyeda2kicad:CAP-TH_BD6.3-P2.50-D1.0-FD"
 		(layer "F.Cu")
 		(at 178.2 89.2)
-		(descr "Capacitor SMD 0805 (2012 Metric), square (rectangular) end terminal, IPC-7351 nominal, (Body size source: IPC-SM-782 page 76, https://www.pcb-3d.com/wordpress/wp-content/uploads/ipc-sm-782a_amendment_1_and_2.pdf, https://docs.google.com/spreadsheets/d/1BsfQQcO9C6DZCsRaXUlFlo91Tg2WpOkGARC1WS5S8t0/edit?usp=sharing), generated with kicad-footprint-generator")
-		(tags "capacitor")
 		(property "Reference" "C11"
-			(at 0 -1.68 0)
+			(at 4.05 0.8 90)
 			(layer "F.SilkS")
 			(effects
@@
 		)
 		(property "Value" "100uF"
-			(at 0 1.68 0)
+			(at 0 4 0)
 			(layer "F.Fab")
 			(hide yes)
@@
 		(sheetname "/")
 		(sheetfile "mini-dyno.kicad_sch")
-		(attr smd)
+		(attr through_hole)
 		(fp_line
-			(start -0.261252 -0.735)
-			(end 0.261252 -0.735)
+			(start -1.78 -1.52)
+			(end -0.76 -1.52)
 			(stroke
-				(width 0.12)
+				(width 0.25)
 				(type solid)
 			)
@@
 		)
 		(fp_line
-			(start -0.261252 0.735)
-			(end 0.261252 0.735)
+			(start -1.27 -2.03)
+			(end -1.27 -1.02)
 			(stroke
-				(width 0.12)
+				(width 0.25)
 				(type solid)
 			)
 			(layer "F.SilkS")
 		)
-		(fp_rect
-			(start -1.7 -0.98)
-			(end 1.7 0.98)
+		(fp_circle
+			(center 0 0)
+			(end 3.15 0)
 			(stroke
-				(width 0.05)
+				(width 0.25)
 				(type solid)
 			)
 			(fill no)
-			(layer "F.CrtYd")
+			(layer "F.SilkS")
 		)
-		(fp_rect
-			(start -1 -0.625)
-			(end 1 0.625)
+		(fp_circle
+			(center -3.15 3.15)
+			(end -3.12 3.15)
 			(stroke
-				(width 0.1)
+				(width 0.06)
+				(type solid)
+			)
+			(fill no)
+			(layer "F.Fab")
+		)
+		(fp_circle
+			(center -1.27 0)
+			(end -1.12 0)
+			(stroke
+				(width 0.3)
+				(type solid)
+			)
+			(fill no)
+			(layer "F.Fab")
+		)
+		(fp_circle
+			(center 1.27 0)
+			(end 1.42 0)
+			(stroke
+				(width 0.3)
 				(type solid)
 			)
@@
 			(effects
 				(font
-					(size 0.5 0.5)
-					(thickness 0.08)
+					(size 1 1)
+					(thickness 0.15)
 				)
 			)
 		)
-		(pad "1" smd roundrect
-			(at -0.95 0)
-			(size 1 1.45)
-			(layers "F.Cu" "F.Mask" "F.Paste")
-			(roundrect_rratio 0.25)
+		(pad "1" thru_hole circle
+			(at -1.27 0)
+			(size 1.6 1.6)
+			(drill 0.999998)
+			(layers "*.Cu" "*.Mask")
+			(remove_unused_layers no)
 			(net 2 "GND")
 			(pintype "passive")
 		)
-		(pad "2" smd roundrect
-			(at 0.95 0)
-			(size 1 1.45)
-			(layers "F.Cu" "F.Mask" "F.Paste")
-			(roundrect_rratio 0.25)
+		(pad "2" thru_hole circle
+			(at 1.27 0)
+			(size 1.6 1.6)
+			(drill 0.999998)
+			(layers "*.Cu" "*.Mask")
+			(remove_unused_layers no)
 			(net 4 "+5V")
 			(pintype "passive")
 		)
 		(embedded_fonts no)
-		(model "${KICAD9_3DMODEL_DIR}/Capacitor_SMD.3dshapes/C_0805_2012Metric.step"
+		(model "${EASYEDA2KICAD}/easyeda2kicad.3dshapes/CAP-TH_BD6.3-P2.50-D1.0-FD.wrl"
 			(offset
-				(xyz 0 0 0)
+				(xyz 0 -0 0)
 			)
 			(scale
@@
 		(descr "LED, diameter 5.0mm, 2 pins, http://cdn-reichelt.de/documents/datenblatt/A500/LL-504BC2E-009.pdf, generated by kicad-footprint-generator")
 		(tags "LED")
-		(property "Reference" "POWER"
+		(property "Reference" "D3"
 			(at 1.27 -3.96 90)
 			(layer "F.SilkS")
@@
 	(footprint "Capacitor_SMD:C_0805_2012Metric"
 		(layer "F.Cu")
-		(at 178.2 92.8)
+		(at 178.2 95)
 		(descr "Capacitor SMD 0805 (2012 Metric), square (rectangular) end terminal, IPC-7351 nominal, (Body size source: IPC-SM-782 page 76, https://www.pcb-3d.com/wordpress/wp-content/uploads/ipc-sm-782a_amendment_1_and_2.pdf, https://docs.google.com/spreadsheets/d/1BsfQQcO9C6DZCsRaXUlFlo91Tg2WpOkGARC1WS5S8t0/edit?usp=sharing), generated with kicad-footprint-generator")
 		(tags "capacitor")
@@
 		(descr "LED, diameter 5.0mm, 2 pins, http://cdn-reichelt.de/documents/datenblatt/A500/LL-504BC2E-009.pdf, generated by kicad-footprint-generator")
 		(tags "LED")
-		(property "Reference" "STATUS"
+		(property "Reference" "D4"
 			(at 1.27 -3.96 90)
 			(layer "F.SilkS")
@@
 	)
 	(segment
-		(start 179.15 94.69)
-		(end 178.2 95.64)
-		(width 1)
-		(layer "F.Cu")
-		(net 4)
-	)
-	(segment
 		(start 173.7 81.8)
 		(end 175.6 83.7)
@@
 	)
 	(segment
-		(start 179.15 92.8)
-		(end 179.15 94.69)
+		(start 179.15 96.69)
+		(end 179.15 95)
 		(width 1)
 		(layer "F.Cu")
@@
 	)
 	(segment
-		(start 179.15 89.2)
-		(end 179.15 84.11)
+		(start 179.15 89.52)
+		(end 179.47 89.2)
 		(width 1)
 		(layer "F.Cu")
@@
 	)
 	(segment
-		(start 179.15 92.8)
-		(end 179.15 89.2)
-		(width 1)
+		(start 173.7 80.5)
+		(end 173.7 81.8)
+		(width 0.6)
 		(layer "F.Cu")
 		(net 4)
 	)
 	(segment
-		(start 173.7 80.5)
-		(end 173.7 81.8)
-		(width 0.6)
+		(start 178.2 97.64)
+		(end 179.15 96.69)
+		(width 1)
 		(layer "F.Cu")
 		(net 4)
@@
 	)
 	(segment
-		(start 188.2 94.6)
-		(end 179.24 94.6)
+		(start 185.16 97.64)
+		(end 188.2 94.6)
 		(width 1)
 		(layer "F.Cu")
@@
 	)
 	(segment
-		(start 179.24 94.6)
-		(end 178.2 95.64)
+		(start 178.2 97.64)
+		(end 185.16 97.64)
 		(width 1)
 		(layer "F.Cu")
@@
 	)
 	(segment
+		(start 179.6 83.66)
+		(end 179.6 89.07)
+		(width 1)
+		(layer "F.Cu")
+		(net 4)
+	)
+	(segment
+		(start 179.15 95)
+		(end 179.15 89.52)
+		(width 1)
+		(layer "F.Cu")
+		(net 4)
+	)
+	(segment
 		(start 175.64 83.66)
 		(end 175.6 83.7)
 		(width 1)
 		(layer "F.Cu")
+		(net 4)
+	)
+	(segment
+		(start 179.6 89.07)
+		(end 179.47 89.2)
+		(width 1)
+		(layer "F.Cu")

Commit message: Update PCB
Parts:
- C11: value 100uF -> 35ZLH100MEFC6.3X11
- moved C11 0.16 mm to (178.1, 89.3), turned to 180 degrees
Connections:
- C11 pad 1: GND -> +5V
- C11 pad 2: +5V -> GND
Changed lines of the file:
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@@
+		)
+	)
+	(footprint "easyeda2kicad:CAP-TH_BD6.3-P2.50-D1.0-FD"
+		(layer "F.Cu")
+		(at 178.07 89.3 180)
+		(property "Reference" "C11"
+			(at -4.23 -0.3 90)
+			(layer "F.SilkS")
+			(effects
+				(font
+					(size 1 1)
+					(thickness 0.15)
+				)
+			)
+		)
+		(property "Value" "35ZLH100MEFC6.3X11"
+			(at 0 4 0)
+			(layer "F.Fab")
+			(effects
+				(font
+					(size 1 1)
+					(thickness 0.15)
+				)
+			)
+		)
+		(property "Datasheet" "https://lcsc.com/product-detail/Aluminum-Electrolytic-Capacitors-Leaded_Rubycon_35ZLH100MEFC6-3X1_100uF-107-20-35V_C109392.html"
+			(at 0 0 0)
+			(layer "F.Fab")
+			(hide yes)
+			(effects
+				(font
+					(size 1.27 1.27)
+					(thickness 0.15)
+				)
+			)
+		)
+		(property "Description" ""
+			(at 0 0 0)
+			(layer "F.Fab")
+			(hide yes)
+			(effects
+				(font
+					(size 1.27 1.27)
+					(thickness 0.15)
+				)
+			)
+		)
+		(property "LCSC Part" "C109392"
+			(at 0 0 180)
+			(unlocked yes)
+			(layer "F.Fab")
+			(hide yes)
+			(effects
+				(font
+					(size 1 1)
+					(thickness 0.15)
+				)
+			)
+		)
+		(sheetname "/")
+		(sheetfile "mini-dyno.kicad_sch")
+		(attr through_hole)
+		(fp_line
+			(start -1.27 -2.03)
+			(end -1.27 -1.02)
+			(stroke
+				(width 0.25)
+				(type solid)
+			)
+			(layer "F.SilkS")
+		)
+		(fp_line
+			(start -1.78 -1.52)
+			(end -0.76 -1.52)
+			(stroke
+				(width 0.25)
+				(type solid)
+			)
+			(layer "F.SilkS")
+		)
+		(fp_circle
+			(center 0 0)
+			(end 3.15 0)
+			(stroke
+				(width 0.25)
+				(type solid)
+			)
+			(fill no)
+			(layer "F.SilkS")
+		)
+		(fp_circle
+			(center 1.27 0)
+			(end 1.42 0)
+			(stroke
+				(width 0.3)
+				(type solid)
+			)
+			(fill no)
+			(layer "F.Fab")
+		)
+		(fp_circle
+			(center -1.27 0)
+			(end -1.12 0)
+			(stroke
+				(width 0.3)
+				(type solid)
+			)
+			(fill no)
+			(layer "F.Fab")
+		)
+		(fp_circle
+			(center -3.15 3.15)
+			(end -3.12 3.15)
+			(stroke
+				(width 0.06)
+				(type solid)
+			)
+			(fill no)
+			(layer "F.Fab")
+		)
+		(fp_text user "${REFERENCE}"
+			(at 0 0 0)
+			(layer "F.Fab")
+			(effects
+				(font
+					(size 1 1)
+					(thickness 0.15)
+				)
+			)
+		)
+		(pad "1" thru_hole circle
+			(at -1.27 0 180)
+			(size 1.6 1.6)
+			(drill 0.999998)
+			(layers "*.Cu" "*.Mask")
+			(remove_unused_layers no)
+			(net 4 "+5V")
+			(pinfunction "1")
+			(pintype "input")
+		)
+		(pad "2" thru_hole circle
+			(at 1.27 0 180)
+			(size 1.6 1.6)
+			(drill 0.999998)
+			(layers "*.Cu" "*.Mask")
+			(remove_unused_layers no)
+			(net 2 "GND")
+			(pinfunction "2")
+			(pintype "input")
+		)
+		(embedded_fonts no)
+		(model "${EASYEDA2KICAD}/easyeda2kicad.3dshapes/CAP-TH_BD6.3-P2.50-D1.0-FD.wrl"
+			(offset
+				(xyz 0 -0 0)
+			)
+			(scale
+				(xyz 1 1 1)
+			)
+			(rotate
+				(xyz 0 0 0)
+			)
 		)
 	)
@@
 			)
 			(scale
-				(xyz 1 1 1)
-			)
-			(rotate
-				(xyz 0 0 0)
-			)
-		)
-	)
-	(footprint "easyeda2kicad:CAP-TH_BD6.3-P2.50-D1.0-FD"
-		(layer "F.Cu")
-		(at 178.2 89.2)
-		(property "Reference" "C11"
-			(at 4.05 0.8 90)
-			(layer "F.SilkS")
-			(effects
-				(font
-					(size 1 1)
-					(thickness 0.15)
-				)
-			)
-		)
-		(property "Value" "100uF"
-			(at 0 4 0)
-			(layer "F.Fab")
-			(hide yes)
-			(effects
-				(font
-					(size 1 1)
-					(thickness 0.15)
-				)
-			)
-		)
-		(property "Datasheet" "~"
-			(at 0 0 0)
-			(layer "F.Fab")
-			(hide yes)
-			(effects
-				(font
-					(size 1.27 1.27)
-					(thickness 0.15)
-				)
-			)
-		)
-		(property "Description" "Unpolarized capacitor"
-			(at 0 0 0)
-			(layer "F.Fab")
-			(hide yes)
-			(effects
-				(font
-					(size 1.27 1.27)
-					(thickness 0.15)
-				)
-			)
-		)
-		(property ki_fp_filters "C_*")
-		(sheetname "/")
-		(sheetfile "mini-dyno.kicad_sch")
-		(attr through_hole)
-		(fp_line
-			(start -1.78 -1.52)
-			(end -0.76 -1.52)
-			(stroke
-				(width 0.25)
-				(type solid)
-			)
-			(layer "F.SilkS")
-		)
-		(fp_line
-			(start -1.27 -2.03)
-			(end -1.27 -1.02)
-			(stroke
-				(width 0.25)
-				(type solid)
-			)
-			(layer "F.SilkS")
-		)
-		(fp_circle
-			(center 0 0)
-			(end 3.15 0)
-			(stroke
-				(width 0.25)
-				(type solid)
-			)
-			(fill no)
-			(layer "F.SilkS")
-		)
-		(fp_circle
-			(center -3.15 3.15)
-			(end -3.12 3.15)
-			(stroke
-				(width 0.06)
-				(type solid)
-			)
-			(fill no)
-			(layer "F.Fab")
-		)
-		(fp_circle
-			(center -1.27 0)
-			(end -1.12 0)
-			(stroke
-				(width 0.3)
-				(type solid)
-			)
-			(fill no)
-			(layer "F.Fab")
-		)
-		(fp_circle
-			(center 1.27 0)
-			(end 1.42 0)
-			(stroke
-				(width 0.3)
-				(type solid)
-			)
-			(fill no)
-			(layer "F.Fab")
-		)
-		(fp_text user "${REFERENCE}"
-			(at 0 0 0)
-			(layer "F.Fab")
-			(effects
-				(font
-					(size 1 1)
-					(thickness 0.15)
-				)
-			)
-		)
-		(pad "1" thru_hole circle
-			(at -1.27 0)
-			(size 1.6 1.6)
-			(drill 0.999998)
-			(layers "*.Cu" "*.Mask")
-			(remove_unused_layers no)
-			(net 2 "GND")
-			(pintype "passive")
-		)
-		(pad "2" thru_hole circle
-			(at 1.27 0)
-			(size 1.6 1.6)
-			(drill 0.999998)
-			(layers "*.Cu" "*.Mask")
-			(remove_unused_layers no)
-			(net 4 "+5V")
-			(pintype "passive")
-		)
-		(embedded_fonts no)
-		(model "${EASYEDA2KICAD}/easyeda2kicad.3dshapes/CAP-TH_BD6.3-P2.50-D1.0-FD.wrl"
-			(offset
-				(xyz 0 -0 0)
-			)
-			(scale

Commit message: Update PCB
Parts:
- removed D5: SS310_C14281, easyeda2kicad:SMB_L4.6-W3.6-LS5.3-RD
- removed USB3: MC-710A, easyeda2kicad:USB-C-TH_MC-710A
- added H1: ~, MountingHole:MountingHole_3.2mm_M3_Pad, F.Cu at (123.0, 72.0)
- added H2: ~, MountingHole:MountingHole_3.2mm_M3_Pad, F.Cu at (183.0, 72.0)
- added H3: ~, MountingHole:MountingHole_3.2mm_M3_Pad, F.Cu at (183.0, 107.0)
- added H4: ~, MountingHole:MountingHole_3.2mm_M3_Pad, F.Cu at (123.0, 107.0)
- added Q1: AO3400A, Package_TO_SOT_SMD:SOT-23_Handsoldering, F.Cu at (179.8, 132.8)
- added R17: 1kΩ, Resistor_SMD:R_0805_2012Metric, F.Cu at (109.3, 117.1)
- added R18: 5.1kΩ, Resistor_SMD:R_0805_2012Metric, F.Cu at (109.3, 120.0)
- added R19: 5.1kΩ, Resistor_SMD:R_0805_2012Metric, F.Cu at (109.3, 123.0)
- added R20: 1MΩ, Resistor_SMD:R_0805_2012Metric, F.Cu at (131.4, 126.3)
- added TP1: VBUS, TestPoint:TestPoint_THTPad_2.0x2.0mm_Drill1.0mm, F.Cu at (100.2, 99.3)
- added TP2: 5V, TestPoint:TestPoint_THTPad_2.0x2.0mm_Drill1.0mm, F.Cu at (99.9, 89.1)
- added TP3: 3V3, TestPoint:TestPoint_THTPad_2.0x2.0mm_Drill1.0mm, F.Cu at (98.3, 79.9)
- added TP4: 5V_MOTOR, TestPoint:TestPoint_THTPad_2.0x2.0mm_Drill1.0mm, F.Cu at (105.8, 81.9)
- added TP5: GND, TestPoint:TestPoint_THTPad_2.0x2.0mm_Drill1.0mm, F.Cu at (105.8, 74.8)
- added U3: ESP32-C3-MINI-1, PCM_Espressif:ESP32-C3-MINI-1, F.Cu at (144.0, 108.5)
- added USB2: DATA, easyeda2kicad:USC-C-SMD_USB4085-GF-A, F.Cu at (124.0, 97.0)
- C10, C2, C4, C7: value 0.1uF -> 10uF
- C11: value 35ZLH100MEFC6.3X11 -> 0.1uF; footprint easyeda2kicad:CAP-TH_BD6.3-P2.50-D1.0-FD -> Capacitor_SMD:C_0805_2012Metric
- C3: value 1uF -> 0.1uF
- C6, C8: value 10uF -> 0.1uF
- C9: value 10uF -> 1uF
- D1: value ESD122DMYR -> D_TVS; footprint easyeda2kicad:X2SON-3_L1.3-W0.6-L -> Diode_SMD:D_SMB
- D2: value SMBJ5.0A_C83333 -> D_Schottky; footprint easyeda2kicad:SMB_L4.6-W3.6-LS5.3-RD -> Diode_SMD:D_SMB
- F1: value TLC-PSML400 -> Polyfuse; footprint easyeda2kicad:F0805 -> Fuse:Fuse_0805_2012Metric_Pad1.15x1.40mm_HandSolder
- R1: value 10kΩ -> 5.1kΩ
- R10: value 1MΩ -> 10kΩ
- R11, R5: value 10kΩ -> 100Ω
- R12, R14, R15: value 100Ω -> 10kΩ
- R13, R6, R7: value 10kΩ -> 0Ω; footprint Resistor_SMD:R_0805_2012Metric -> Resistor_SMD:R_1206_3216Metric_Pad1.30x1.75mm_HandSolder
- R16: value 100Ω -> 1kΩ
- R3: value 5.1kΩ -> 0Ω; footprint Resistor_SMD:R_0805_2012Metric -> Resistor_SMD:R_1206_3216Metric_Pad1.30x1.75mm_HandSolder
- R4: value 5.1kΩ -> 100Ω
- R9: value 5.1kΩ -> 10kΩ
- U1: value ESP32-C3-MINI-1 -> AZ1117IH-3.3TRG1; footprint PCM_Espressif:ESP32-C3-MINI-1 -> easyeda2kicad:SOT-223-4_L6.5-W3.5-P2.30-LS7.0-BR
- U2: value TLV75733PDBVR -> HX711; footprint easyeda2kicad:SOT-23-5_L2.9-W1.6-P0.95-LS2.8-BL -> easyeda2kicad:SOP-16_L10.0-W3.9-P1.27-LS6.0-BL
- U4: value HX711_C6705483 -> TPD2S017; footprint easyeda2kicad:SOP-16_L10.0-W3.9-P1.27-LS6.0-BL -> Package_TO_SOT_SMD:SOT-23-6
- USB1: value MC-710A -> POWER; footprint easyeda2kicad:USB-C-TH_MC-710A -> easyeda2kicad:USC-C-SMD_USB4085-GF-A
- moved R4 98.8 mm to (96.1, 123.0)
- moved R8 81.6 mm to (110.1, 109.0), turned to 0 degrees
- moved R2 78.8 mm to (108.7, 98.9), turned to 180 degrees
- moved R12 76.4 mm to (104.9, 117.1), turned to 0 degrees
- moved R14 74.0 mm to (104.9, 123.0)
- moved C6 70.7 mm to (118.2, 117.2)
- moved R1 66.6 mm to (105.8, 92.6)
- moved C5 64.2 mm to (118.2, 114.2)
- moved C3 63.7 mm to (113.8, 120.2), turned to 0 degrees
- moved C8 63.5 mm to (118.2, 123.2), turned to 0 degrees
- moved C11 63.5 mm to (122.7, 120.2), turned to 0 degrees
- moved C12 62.3 mm to (122.7, 123.2)
- moved R13 61.8 mm to (186.1, 121.2), turned to 180 degrees
- moved C2 61.3 mm to (113.8, 117.2)
- moved R15 60.5 mm to (104.9, 126.0)
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Connections:
- C1 pad 1: +3V3 -> Net-(U1-INPUT)
- C10 pad 1: Net-(U4-INPA) -> GND
- C10 pad 2: Net-(U4-INNA) -> Net-(D2-K)
- C11 pad 1: +5V -> GND
- C11 pad 2: GND -> Net-(D2-K)
- C12 pad 1: GND -> +3V3
- C12 pad 2: +5V -> GND
- C2 pad 1: +3V3 -> GND
- C2 pad 2: GND -> Net-(J1-Pin_1)
- C3 pad 1: GND -> Net-(U2-INPA)
- C3 pad 2: Net-(U1-EN/CHIP_PU) -> Net-(U2-INNA)
- C4 pad 1: GND -> Net-(U1-OUTPUT)
- C4 pad 2: Net-(C4-Pad2) -> GND
- C5 pad 2: +5V -> Net-(U2-DVDD)
- C6 pad 2: +3V3 -> Net-(C6-Pad2)
- C8 pad 1: GND -> +3V3
- C8 pad 2: +3V3 -> GND
- C9 pad 2: Net-(J1-Pin_1) -> Net-(U3-EN/CHIP_PU)
- D1 pad 1: GND -> +5V
- D1 pad 2: Net-(D1-IO1) -> GND
- D2 pad 1: +5V -> Net-(D2-K)
- D2 pad 2: GND -> /MOTOR_DRAIN
- F1 pad 1: Net-(F1-Pad1) -> /VBUS
- MOTOR1 pad 1: +5V -> Net-(D2-K)
- MOTOR1 pad 4: GND -> /MOTOR_DRAIN
- R1 pad 1: +3V3 -> GND
- R1 pad 2: Net-(U1-EN/CHIP_PU) -> /CC1_P
- R10 pad 1: GND -> +3V3
- R10 pad 2: Net-(R10-Pad2) -> Net-(U3-EN/CHIP_PU)
- R11 pad 1: Net-(U1-GPIO9) -> /FET_GATE
- R11 pad 2: +3V3 -> Net-(Q1-G)
- R12 pad 1: +3V3 -> GND
- R12 pad 2: Net-(D3-A) -> Net-(Q1-G)
- R13 pad 1: /GPIO10 -> Net-(D2-K)
- R13 pad 2: +3V3 -> +5V
- R14 pad 1: /GPIO5 -> /GPIO10
- R14 pad 2: Net-(D4-A) -> +3V3
- R15 pad 1: Net-(J1-Pin_3) -> Net-(U3-GPIO9)
- R15 pad 2: Net-(U4-INNA) -> +3V3
- R16 pad 1: Net-(J1-Pin_4) -> +3V3
- R16 pad 2: Net-(U4-INPA) -> Net-(D3-A)
- R2 pad 2: Net-(USB3-CC1) -> /CC2_P
- R3 pad 1: GND -> Net-(U1-INPUT)
- R3 pad 2: Net-(USB1-CC1) -> +5V
- R4 pad 1: GND -> Net-(J1-Pin_3)
- R4 pad 2: Net-(USB3-CC2) -> Net-(U2-INNA)
- R5 pad 1: Net-(U1-GPIO19/USB_D+) -> Net-(J1-Pin_4)
- R5 pad 2: Net-(D1-IO1) -> Net-(U2-INPA)
- R6 pad 1: Net-(U1-GPIO18/USB_D-) -> Net-(U2-DVDD)
- R6 pad 2: Net-(D1-IO2) -> +3V3
- R7 pad 1: Net-(C4-Pad2) -> +3V3
- R7 pad 2: Net-(U1-EN/CHIP_PU) -> Net-(U1-OUTPUT)
- R9 pad 1: GND -> Net-(C6-Pad2)
- R9 pad 2: Net-(USB1-CC2) -> Net-(U3-EN/CHIP_PU)
- SW1 pad 2: Net-(C4-Pad2) -> Net-(C6-Pad2)
- U1 pad 2: GND -> Net-(U1-OUTPUT)
- U1 pad 3: +3V3 -> Net-(U1-INPUT)
- U1 pad 4: unconnected-(U1-NC-Pad4) -> Net-(U1-OUTPUT)
- U2 pad 1: +5V -> Net-(U2-DVDD)
- U2 pad 2: GND -> unconnected-(U2-BASE-Pad2)
- U2 pad 3: +5V -> Net-(J1-Pin_1)
- U2 pad 4: unconnected-(U2-NC-Pad4) -> GND
- U2 pad 5: +3V3 -> GND
- U4 pad 1: +3V3 -> /D+
- U4 pad 2: unconnected-(U4-BASE-Pad2) -> GND
- U4 pad 3: Net-(J1-Pin_1) -> /ESD_D+
- U4 pad 4: GND -> /ESD_D-
- U4 pad 5: GND -> +5V
- U4 pad 6: GND -> /D-
- USB1 pad A4: unconnected-(USB1-VBUS-PadA4) -> /VBUS
- USB1 pad A5: Net-(USB1-CC1) -> /CC1_P
- USB1 pad A6: Net-(D1-IO1) -> unconnected-(USB1-Dp1-PadA6)
- USB1 pad A7: Net-(D1-IO2) -> unconnected-(USB1-Dn1-PadA7)
- USB1 pad A9: unconnected-(USB1-VBUS-PadA9) -> /VBUS
- USB1 pad B4: unconnected-(USB1-VBUS-PadB4) -> /VBUS
- USB1 pad B5: Net-(USB1-CC2) -> /CC2_P
- USB1 pad B9: unconnected-(USB1-VBUS-PadB9) -> /VBUS
Routing:
- net +3V3: track 119.1 -> 0.00 mm
- net /GPIO10: track 57.0 -> 0.00 mm, vias 2 -> 0
- net Net-(U1-EN/CHIP_PU): track 47.6 -> 0.00 mm, vias 2 -> 0
- net +5V: track 42.6 -> 0.00 mm
- net Net-(F1-Pad1): track 28.9 -> 0.00 mm
- net /GPIO5: track 28.0 -> 0.00 mm, vias 2 -> 0
- net Net-(J1-Pin_1): track 27.7 -> 0.00 mm, vias 2 -> 0
- net Net-(USB1-CC2): track 24.9 -> 0.00 mm, vias 2 -> 0
- net Net-(U1-GPIO9): track 23.9 -> 0.00 mm, vias 2 -> 0
- net Net-(D1-IO2): track 22.9 -> 0.00 mm, vias 2 -> 0
- net Net-(D1-IO1): track 22.7 -> 0.00 mm
- net GND: track 28.9 -> 7.05 mm, vias 25 -> 2
- net Net-(USB3-CC1): track 16.9 -> 0.00 mm, vias 2 -> 0
- net Net-(C4-Pad2): track 14.6 -> 0.00 mm
- net Net-(U4-INNA): track 12.3 -> 0.00 mm
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- added copper zone on In2.Cu, net +3V3
- added copper zone on In1.Cu, net GND
Other:
- board size 65 x 37 mm -> 70 x 45 mm
- copper layers 2 -> 4
- rule solder_mask_min_width: 0.12 -> 0.1016
- board text removed: "BOOT"
- board text removed: "BY SAM EHLERS"
- board text removed: "D - +"
- board text removed: "DATA"
- board text removed: "DYNO CONTROL"
- board text removed: "E+ E- S- S+"
- board text removed: "MOTOR"
- board text removed: "POWER"
- board text removed: "RESET"

Commit message: Update PCB Layout
Parts:
- TP4: value 5V_MOTOR -> MOTOR
- moved R14 80.1 mm to (178.5, 91.3)
- moved TP3 79.3 mm to (176.9, 69.3)
- moved D1 77.5 mm to (136.0, 72.2)
- moved MOTOR1 75.0 mm to (168.0, 76.0), turned to -90 degrees
- moved TP5 71.1 mm to (176.9, 73.8)
- moved R16 68.6 mm to (173.3, 89.3), turned to -90 degrees
- moved F1 67.2 mm to (130.5, 74.5)
- moved R13 66.6 mm to (143.1, 70.3)
- moved C4 66.0 mm to (155.4, 76.0), turned to 90 degrees
- moved C11 61.3 mm to (156.9, 69.3), turned to -90 degrees
- moved R9 60.3 mm to (153.1, 93.6), turned to 180 degrees
- moved D2 59.9 mm to (161.2, 74.3), turned to -90 degrees
- moved R17 58.9 mm to (163.8, 94.7), turned to 180 degrees
- moved R10 58.2 mm to (153.1, 101.0), turned to 180 degrees
- moved C1 57.5 mm to (141.4, 75.7), turned to 90 degrees
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- renumbered SW1 to Boot, SW2 to Reset
Connections:
- U4 pad 5: +5V -> +3V3
Routing:
- net Net-(J1-Pin_4): track 0.00 -> 52.9 mm, vias 0 -> 2
- net /FET_GATE: track 0.00 -> 50.3 mm, vias 0 -> 2
- net Net-(J1-Pin_1): track 0.00 -> 48.8 mm, vias 0 -> 2
- net Net-(J1-Pin_3): track 0.00 -> 46.5 mm, vias 0 -> 2
- net +3V3: track 0.00 -> 43.0 mm, vias 0 -> 10
- net /GPIO10: track 0.00 -> 40.4 mm, vias 0 -> 2
- net /VBUS: track 0.00 -> 35.3 mm
- net Net-(D2-K): track 0.00 -> 32.2 mm
- net /GPIO5: track 0.00 -> 27.4 mm, vias 0 -> 2
- net /CC2_P: track 0.00 -> 26.0 mm, vias 0 -> 2
- net /CC2: track 0.00 -> 25.8 mm
- net Net-(R8-Pad2): track 0.00 -> 22.1 mm, vias 0 -> 1
- net Net-(C6-Pad2): track 0.00 -> 21.3 mm
- net GND: track 7.05 -> 27.8 mm, vias 2 -> 118
- net Net-(R20-Pad1): track 0.00 -> 20.4 mm
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
Commit message: Update Layout
Routing:
- net GND: vias 118 -> 121
Changed lines of the file:
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@@
 		(capping no)
 		(filling no)
-		(zone_defaults)
 		(pcbplotparams
 			(layerselection 0x00000000_00000000_55555555_5755f5ff)
@@
 	)
 	(via
+		(at 129.6 101.4)
+		(size 0.6858)
+		(drill 0.3302)
+		(layers "F.Cu" "B.Cu")
+		(free yes)
+		(net "GND")
+	)
+	(via
 		(at 128.4 94)
 		(size 0.6858)
@@
 	)
 	(via
+		(at 134.8 100.3)
+		(size 0.6858)
+		(drill 0.3302)
+		(layers "F.Cu" "B.Cu")
+		(free yes)
+		(net "GND")
+	)
+	(via
 		(at 158.2 78)
 		(size 0.45)
@@
 		(layers "F.Cu" "B.Cu")
 		(free yes)
+		(net "GND")
+	)
+	(via
+		(at 132.6 102.8)
+		(size 0.6858)
+		(drill 0.3302)
+		(layers "F.Cu" "B.Cu")
+		(free yes)

Commit message: New Rust Firware
Routing:
- net GND: vias 121 -> 116
Other:
- board text added: "DESIGNED BY"
- board text added: "SAM EHLERS"
Changed lines of the file:
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@@
 			(outputformat 1)
 			(mirror no)
-			(drillshape 1)
+			(drillshape 0)
 			(scaleselection 1)
-			(outputdirectory "")
+			(outputdirectory "../../../gerbers/")
 		)
 	)
@@
 		(layer "Edge.Cuts")
 	)
+	(gr_text "DESIGNED BY"
+		(at 177.8 111.2 90)
+		(layer "F.SilkS")
+		(effects
+			(font
+				(size 0.8128 0.8128)
+				(thickness 0.1524)
+				(bold yes)
+			)
+			(justify left bottom)
+		)
+	)
+	(gr_text "SAM EHLERS"
+		(at 179.2 111.2 90)
+		(layer "F.SilkS")
+		(effects
+			(font
+				(size 0.8128 0.8128)
+				(thickness 0.1524)
+				(bold yes)
+			)
+			(justify left bottom)
+		)
+	)
 	(segment
 		(start 126.16 84.98)
@@
 	)
 	(via
-		(at 177.6 107.4)
-		(size 0.45)
-		(drill 0.2)
-		(layers "F.Cu" "B.Cu")
-		(free yes)
-		(net "GND")
-	)
-	(via
 		(at 147.8 81.3)
 		(size 0.45)
@@
 	)
 	(via
-		(at 176.8 106.1)
-		(size 0.45)
-		(drill 0.2)
-		(layers "F.Cu" "B.Cu")
-		(free yes)
-		(net "GND")
-	)
-	(via
 		(at 145 103.8)
 		(size 0.45)
@@
 	)
 	(via
-		(at 176.8 108.8)
-		(size 0.45)
-		(drill 0.2)
-		(layers "F.Cu" "B.Cu")
-		(free yes)
-		(net "GND")
-	)
-	(via
 		(at 150.4 81.3)
 		(size 0.45)
@@
 	)
 	(via
-		(at 178.4 108.8)
-		(size 0.45)
-		(drill 0.2)
-		(layers "F.Cu" "B.Cu")
-		(free yes)
-		(net "GND")
-	)
-	(via
 		(at 131.8 69.4)
 		(size 0.45)
@@
 		(size 0.45)
 		(drill 0.2)
-		(layers "F.Cu" "B.Cu")
-		(free yes)
-		(net "GND")
-	)
-	(via
-		(at 176 107.4)
-		(size 0.45)
-		(drill 0.2)
